File: hardware/raptor.kicad_pcb (KiCad board)
At the start: 4 copper layers, 22.7 x 74 mm, 72 parts, among them IC1 RAPTORQFN56, IC2 FT232H, IC3 MCP1755, IC4 93C56, J1 USB, J10 CONN_02, J11 CONN_20, J12 CONN_20, J2 CONN_03, J3 CONN_03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

Commit message: Add files via upload
Parts:
- removed C12, C13, C23: 2.2uf, Capacitor_SMD:C_0603_1608Metric
- removed C24, C6: 27pf, Capacitor_SMD:C_0603_1608Metric
- removed C7: 1uf, Capacitor_SMD:C_0603_1608Metric
- removed J10, J6, J7: CONN_02, Connector_PinHeader_2.54mm:PinHeader_1x02_P2.54mm_Vertical
- removed J4, J5, J8: CONN_03, Connector_PinHeader_2.54mm:PinHeader_1x03_P2.54mm_Vertical
- removed U$1: MCP1316M, Package_TO_SOT_SMD:SOT-23-5
- removed U$3: MCP1501SOT23-6, Package_TO_SOT_SMD:SOT-23-6
- removed U$4: MCP1811, Package_TO_SOT_SMD:SOT-23
- added C3: 0.1uf, Capacitor_SMD:C_0603_1608Metric, F.Cu at (145.4, 127.3)
- added G1: LOGO, raptor-KiCadVersion:logo, F.Cu at (148.8, 92.5)
- added IC5: TMUX1574RSVR, SamacSys_Parts:QFN40P180X260X55-16N, B.Cu at (141.9, 95.8)
- added R11: 10K, Resistor_SMD:R_0603_1608Metric, B.Cu at (143.0, 91.6)
- added R15: 10K, Resistor_SMD:R_0603_1608Metric, F.Cu at (143.1, 101.6)
- added R16: 10K, Resistor_SMD:R_0603_1608Metric, F.Cu at (141.8, 105.4)
- added R22: 10k, Resistor_SMD:R_0603_1608Metric, B.Cu at (154.4, 93.6)
- added R23: 0, Resistor_SMD:R_0603_1608Metric, F.Cu at (155.7, 119.0)
- added R24: 10K, Resistor_SMD:R_0603_1608Metric, B.Cu at (147.4, 132.7)
- added R25: 0, Resistor_SMD:R_0603_1608Metric, F.Cu at (154.8, 127.2)
- added R8: 10K, Resistor_SMD:R_0603_1608Metric, F.Cu at (153.7, 108.8)
- added U1: SN74LVC1G125DCKR, parts and footprints:SOT65P210X110-5N, B.Cu at (147.6, 130.8)
- added U1: MCP1316M, Package_TO_SOT_SMD:SOT-23-5, F.Cu at (153.9, 94.5)
- C1: value 27pf -> 10nf
- C2: value 27pf -> 0.1uf; moved to F.Cu
- J2, J3: value CONN_03 -> Conn_01x02_Male; footprint Connector_PinHeader_2.54mm:PinHeader_1x03_P2.54mm_Vertical -> Connector_PinHeader_2.54mm:PinHeader_1x02_P2.54mm_Vertical
- R10: value 50 -> 10K
- R14, R2: value 4.7K -> 10k
- R9: value 2K 1% -> 12K 1%; moved to F.Cu
- U2: footprint Package_SO:SOIC-8_3.9x4.9mm_P1.27mm -> parts and footprints:SOIC127P790X216-8N
- moved J3 58.7 mm to (154.6, 131.1), turned to 0 degrees
- moved D7 56.3 mm to (146.6, 133.9), turned to 90 degrees
- moved J2 51.3 mm to (142.1, 133.6)
- moved D4 39.2 mm to (142.0, 86.6), turned to 90 degrees
- moved C5 34.1 mm to (143.8, 111.6), turned to 90 degrees
- moved D3 33.1 mm to (151.7, 133.9), turned to 90 degrees
- moved D1 32.7 mm to (148.3, 133.9), turned to 90 degrees
- moved R12 28.9 mm to (141.8, 108.4)
- moved D5 26.1 mm to (148.1, 101.6), turned to 90 degrees
- moved D6 25.7 mm to (146.3, 101.6), turned to 90 degrees
- moved C2 23.8 mm to (149.2, 128.5), turned to 0 degrees
- moved IC3 23.8 mm to (154.4, 99.8), turned to 180 degrees
- moved C4 23.5 mm to (154.7, 102.6)
- moved C9 23.2 mm to (151.4, 101.6), turned to 270 degrees
- moved U2 22.0 mm to (147.4, 106.9), turned to 180 degrees
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Connections:
- C15 pad 2: +3V3 -> VDD
- C16 pad 1: +3V3 -> VDD
- C17 pad 1: +3V3 -> VDD
- C2 pad 1: GND -> VDD
- C2 pad 2: Net-(C1-Pad1) -> GND
- C20 pad 1: +3V3 -> VDD
- C21 pad 1: +3V3 -> VDD
- C5 pad 2: +3V3 -> VDD
- IC1 pad 34: Net-(IC1-Pad34) -> /VREF+
- IC2 pad 12: +3V3 -> VDD
- IC2 pad 2: Net-(C1-Pad1) -> Net-(IC2-Pad2)
- IC2 pad 21: Net-(IC2-Pad21) -> /TMUX_SEL
- IC2 pad 24: +3V3 -> VDD
- IC2 pad 25: Net-(IC2-Pad25) -> /TXD_EN
- IC2 pad 3: +3V3 -> VDD
- IC2 pad 34: Net-(IC2-Pad34) -> Net-(C1-Pad1)
- IC2 pad 39: +3V3 -> VDD
- IC2 pad 40: +5V -> VDD
- IC2 pad 46: +3V3 -> VDD
- IC2 pad 8: +3V3 -> VDD
- IC4 pad 6: +3V3 -> VDD
- J2 pad 1: /RAPTOR_CS -> Net-(J2-Pad1)
- J2 pad 2: Net-(J2-Pad2) -> /TMUX_SEL
- J3 pad 1: /RAPTOR_D1 -> GND
- J3 pad 2: Net-(J3-Pad2) -> /TXD_EN
- R1 pad 1: /RAPTOR_D2 -> VDD
- R1 pad 2: +3V3 -> /RAPTOR_D2
- R10 pad 1: Net-(J8-Pad3) -> VDD
- R10 pad 2: Net-(C12-Pad1) -> /MEM_SO
- R12 pad 1: /RAPTOR_D3 -> VDD
- R12 pad 2: +3V3 -> /RAPTOR_D3
- R13 pad 1: +3V3 -> VDD
- R14 pad 1: Net-(IC2-Pad31) -> VDD
- R14 pad 2: +5V -> Net-(IC2-Pad45)
- R2 pad 1: GND -> VDD
- R2 pad 2: Net-(IC2-Pad31) -> Net-(IC2-Pad44)
- R5 pad 1: Net-(IC2-Pad34) -> Net-(C1-Pad1)
- R5 pad 2: +3V3 -> VDD
- R6 pad 1: +3V3 -> VDD
- RESET1 pad 1: Net-(R4-Pad1) -> GND
- RESET1 pad 2: Net-(R4-Pad1) -> GND
- RESET1 pad 3: GND -> Net-(R4-Pad1)
- RESET1 pad 4: GND -> Net-(R4-Pad1)
- RESET1 pad 5: (no net) -> GND
- U2 pad 1: Net-(J2-Pad2) -> /MEM_CS
- U2 pad 2: Net-(J3-Pad2) -> /MEM_SO
- U2 pad 5: Net-(J5-Pad2) -> /MEM_SI
- U2 pad 6: Net-(J4-Pad2) -> /MEM_SCK
- U2 pad 8: +3V3 -> VDD
- X1 pad 1: Net-(C1-Pad1) -> Net-(IC2-Pad1)
- X1 pad 3: Net-(IC2-Pad1) -> Net-(IC2-Pad2)
Routing:
- net VDD: track 0.00 -> 280.0 mm, vias 0 -> 14
- net GND: track 0.00 -> 237.6 mm, vias 0 -> 18
- net /P1: track 0.00 -> 83.1 mm, vias 0 -> 2
- net /P3: track 0.00 -> 79.7 mm, vias 0 -> 4
- net /P0: track 0.00 -> 72.9 mm, vias 0 -> 2
- net /P2: track 0.00 -> 56.1 mm, vias 0 -> 2
- net /TXD_EN: track 0.00 -> 56.0 mm, vias 0 -> 2
- net /MSI1: track 0.00 -> 55.3 mm, vias 0 -> 3
- net /SDA: track 0.00 -> 54.1 mm, vias 0 -> 3
- net /RAPTOR_D1: track 0.00 -> 51.7 mm, vias 0 -> 3
- net Net-(J2-Pad1): track 0.00 -> 51.2 mm
- net /MEM_SI: track 0.00 -> 50.1 mm, vias 0 -> 1
- net /MSO0: track 0.00 -> 49.7 mm, vias 0 -> 2
- net /TMUX_SEL: track 0.00 -> 47.3 mm
- net /RAPTOR_D0: track 0.00 -> 46.4 mm, vias 0 -> 3
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- removed copper zone on Route15, net GND
- removed copper zone on Route2, net GND
Other:
- board size 22.7 x 74 mm -> 22.9 x 57.7 mm
- net class Default: trace_width 0.1524 -> 0.1016
- rule trace_min: 0.1524 -> 0.1016
- board text added: "P6"
- board text added: "P7"
- board text removed: "+5V"
- board text removed: "P6>"
- board text removed: "P7>"
- board text removed: "RX0<"
- board text removed: "TX0<"
- board text removed: "TX1>"
- board text removed: "VREF+<"
- board text removed: "rCS"
- board text removed: "rD0"
- board text removed: "rD1"
- board text removed: "rSCK"
- board text removed: "usbCs"
- board text removed: "usbS0Rxd<>"
- board text removed: "usbSckTxd<>"
- board text removed: "usbSi"

Commit message: Add files via upload
Parts:
- G1: moved to B.Cu
- moved G1 29.3 mm to (148.6, 121.8), turned to 180 degrees
Other:
- board text added: "+5V"
- board text added: "<C1"
- board text added: "<GND"
- board text added: "C0>"
- board text added: "TMUX_SEL"
- board text added: "TX1>"
- board text added: "TXD_EN"
- board text removed: "1.c"
- board text removed: "C0"
- board text removed: "C1"
- board text removed: "GND"

Commit message: Add files via upload
Parts:
- G1: moved to F.Cu
- moved G1 24.4 mm to (149.5, 97.4), turned to 0 degrees
- moved C21 1.23 mm to (155.2, 106.9), turned to 270 degrees
- moved J1 0.81 mm to (148.3, 88.6)
- moved C15 0.45 mm to (155.2, 103.7), turned to 270 degrees
- moved FUSE_0 0.09 mm to (146.8, 87.5)
- moved X1 0.06 mm to (154.5, 99.3)
Routing:
- net GND: track 237.6 -> 243.2 mm, vias 18 -> 19
- net /TXD_EN: track 56.0 -> 51.1 mm, vias 2 -> 4
- net /C1: track 31.5 -> 29.2 mm
- net Net-(FUSE1-Pad2): track 24.6 -> 26.6 mm
- net VDD: track 280.0 -> 281.3 mm
- net +5V: track 32.2 -> 33.0 mm

Commit message: Add files via upload
Other:
- board text added: "C0"
- board text added: "C1"
- board text added: "GND"
- board text removed: "<C1"
- board text removed: "<GND"
- board text removed: "C0>"
- board text removed: "TX1>"
- board text removed: "pin1"
- board text removed: "pin56"

Commit message: Add files via upload
Parts:
- moved R11 46.0 mm to (138.9, 137.4), turned to 270 degrees
- moved R23 11.8 mm to (146.6, 111.5), turned to 180 degrees
- moved RESET1 2.81 mm to (146.8, 94.7)
- moved IC5 0.66 mm to (142.2, 95.2)
Routing:
- net Net-(J2-Pad1): track 51.3 -> 4.36 mm
- net /MSI1: track 55.3 -> 22.5 mm, vias 3 -> 1
- net /P3: track 79.8 -> 50.6 mm, vias 4 -> 2
- net VDD: track 281.3 -> 252.7 mm, vias 14 -> 13
- net /MEM_SI: track 50.1 -> 26.2 mm, vias 1 -> 2
- net /CS0: track 38.4 -> 58.7 mm
- net /P1: track 83.1 -> 63.3 mm
- net /RX0: track 4.07 -> 21.0 mm, vias 0 -> 2
- net /SCK0: track 45.2 -> 29.5 mm, vias 2 -> 1
- net Net-(FUSE_0-Pad2): track 23.3 -> 38.9 mm, vias 2 -> 1
- net /RAPTOR_D3: track 45.5 -> 31.7 mm
- net /MCS1: track 19.7 -> 33.2 mm
- net /MSO0: track 49.7 -> 36.8 mm, vias 2 -> 1
- net /TX0: track 36.1 -> 23.5 mm, vias 0 -> 1
- net /MEM_SCK: track 17.8 -> 29.8 mm, vias 2 -> 1
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Other:
- net class Default: trace_width 0.1016 -> 0.127
- rule trace_min: 0.1016 -> 0.127

Commit message: update logo and silkscreen (2)
Parts:
- moved G1 4.22 mm to (145.4, 98.5)
- moved R9 1.06 mm to (151.1, 98.0), turned to 270 degrees
Routing:
- net GND: track 245.7 -> 246.9 mm
Other:
- board text added: "PWR"
- board text added: "Rev B"
Changed lines of the file:
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@@
-(kicad_pcb (version 20171130) (host pcbnew "(5.1.4)-1")
+(kicad_pcb (version 20171130) (host pcbnew "(5.1.5-0-10_14)")
   (general
     (thickness 1.6)
-    (drawings 51)
-    (tracks 1788)
+    (drawings 53)
+    (tracks 1790)
     (zones 0)
     (modules 70)
@@
   (layers
     (0 Top signal)
-    (1 Route2 signal)
-    (2 Route15 signal)
-    (31 Bottom signal)
+    (1 Route2 signal hide)
+    (2 Route15 signal hide)
+    (31 Bottom signal hide)
     (32 B.Adhes user hide)
     (33 F.Adhes user hide)
-    (34 B.Paste user)
+    (34 B.Paste user hide)
     (35 F.Paste user hide)
     (36 B.SilkS user hide)
@@
     (38 B.Mask user hide)
     (39 F.Mask user hide)
-    (40 Dwgs.User user)
+    (40 Dwgs.User user hide)
     (41 Cmts.User user hide)
     (42 Eco1.User user hide)
@@
     (44 Edge.Cuts user hide)
     (45 Margin user hide)
-    (46 B.CrtYd user)
-    (47 F.CrtYd user)
+    (46 B.CrtYd user hide)
+    (47 F.CrtYd user hide)
     (48 B.Fab user hide)
     (49 F.Fab user hide)
@@
     (visible_elements 7FFFFFFF)
     (pcbplotparams
-      (layerselection 0x010fc_ffffffff)
+      (layerselection 0x310ff_ffffffff)
       (usegerberextensions true)
       (usegerberattributes false)
@@
       (psa4output false)
       (plotreference true)
-      (plotvalue false)
+      (plotvalue true)
       (plotinvisibletext false)
       (padsonsilk false)
@@
   )
   (module raptor-KiCadVersion:logo (layer Top)
-    (at 149.52 97.37)
+    (at 145.4404 98.4504)
     (attr smd)
     (fp_text reference G1 (at 3.937 -1.651) (layer F.SilkS) hide
@@
   )
   (module Resistor_SMD:R_0603_1608Metric (layer Top)
-    (at 150.42 98.88)
+    (at 151.0792 98.044 270)
     (descr "Resistor SMD 0603 (1608 Metric), square (rectangular) end terminal, IPC_7351 nominal, (Body size source: http://www.tortai-tech.com/upload/download/2011102023233369053.pdf), generated with kicad-footprint-generator")
     (tags resistor)
     (attr smd)
-    (fp_text reference R9 (at 1.7275 0.174 180) (layer F.SilkS)
+    (fp_text reference R9 (at 1.7275 0.174 270) (layer F.SilkS)
       (effects (font (size 0.254 0.254) (thickness 0.0635)))
     )
-    (fp_text value "12K 1%" (at 0 1.43 180) (layer F.Fab)
+    (fp_text value "12K 1%" (at 0 1.43 270) (layer F.Fab)
       (effects (font (size 1 1) (thickness 0.15)))
     )
-    (fp_text user %R (at 0 0 180) (layer F.Fab)
+    (fp_text user %R (at 0 0 270) (layer F.Fab)
       (effects (font (size 0.4 0.4) (thickness 0.06)))
     )
@@
     (fp_line (start -0.8 -0.4) (end 0.8 -0.4) (layer F.Fab) (width 0.1))
     (fp_line (start -0.8 0.4) (end -0.8 -0.4) (layer F.Fab) (width 0.1))
-    (pad 2 smd roundrect (at 0.7875 0) (size 0.875 0.95) (layers Top F.Paste F.Mask) (roundrect_rratio 0.25)
+    (pad 2 smd roundrect (at 0.7875 0 270) (size 0.875 0.95) (layers Top F.Paste F.Mask) (roundrect_rratio 0.25)
       (net 57 "Net-(IC2-Pad5)"))
-    (pad 1 smd roundrect (at -0.7875 0) (size 0.875 0.95) (layers Top F.Paste F.Mask) (roundrect_rratio 0.25)
+    (pad 1 smd roundrect (at -0.7875 0 270) (size 0.875 0.95) (layers Top F.Paste F.Mask) (roundrect_rratio 0.25)
       (net 1 GND))
     (model ${KISYS3DMOD}/Resistor_SMD.3dshapes/R_0603_1608Metric.wrl
@@
     )
   )
+  (gr_text PWR (at 143.3068 87.2236 90) (layer F.SilkS)
+    (effects (font (size 0.6 0.6) (thickness 0.1)))
+  )
+  (gr_text "Rev B" (at 142.0368 127.762) (layer F.SilkS)
+    (effects (font (size 0.6 0.6) (thickness 0.1)))
+  )
   (gr_text TXD_EN (at 152.908 133.858 90) (layer F.SilkS)
     (effects (font (size 0.381 0.381) (thickness 0.09525)))
@@
   )
   (gr_circle (center 154.178 119.888) (end 154.178 119.888) (layer F.SilkS) (width 0.508))
-  (gr_text "RAPTOR EVB" (at 144.61 114.16) (layer F.SilkS)
+  (gr_text "RAPTOR \nEVB" (at 143.6116 115.0112) (layer F.SilkS)
     (effects (font (size 0.75 0.75) (thickness 0.15)))
   )
@@
   (segment (start 150.4026 96.7968) (end 151.0317 96.1677) (width 0.2032) (layer Bottom) (net 1))
   (segment (start 151.0317 96.1677) (end 151.235699 95.963701) (width 0.2032) (layer Bottom) (net 1))
+  (segment (start 151.1555 97.2565) (end 151.892 96.52) (width 0.2032) (layer Top) (net 1))
+  (segment (start 151.0792 97.2565) (end 151.1555 97.2565) (width 0.2032) (layer Top) (net 1))
   (segment (start 140.54388 103.3375) (end 140.53724 103.34414) (width 0.127) (layer Bottom) (net 2))
   (segment (start 142.03 103.3375) (end 140.54388 103.3375) (width 0.127) (layer Bottom) (net 2))

Commit message: Add files via upload
Parts:
- moved G1 4.22 mm to (149.5, 97.4)
- moved R9 1.06 mm to (150.4, 98.9), turned to 0 degrees
Routing:
- net GND: track 246.9 -> 245.7 mm
Other:
- board text removed: "PWR"
- board text removed: "Rev B"

Commit message: recommit previous version
Parts:
- moved G1 4.22 mm to (145.4, 98.5)
- moved R9 1.06 mm to (151.1, 98.0), turned to 270 degrees
Routing:
- net GND: track 245.7 -> 246.9 mm
Other:
- board text added: "PWR"
- board text added: "Rev B"
